Commit message: Update cleanbot.urdf

File: thedush_robots/urdf/cleanbot.urdf (robot description, URDF)
Before this commit: robot mecanum_wheeled_robot, 6 links, 5 joints
Joints:
- joint kinect_joint: origin xyz=0.00128984451294 -0.19538221359 0.084095378876 rpy=0 0 0 -> xyz=0.00128984451294 -0.19538221359 0.084095378876 rpy=0 0 -1.54
